Commit message: ♥ 소나, 리얼센스 관련 interface 변수 선언 빠져있는 부분과  기타 수정

File: tetraDS_description/urdf/tetraDS/tetraDS_bak.xacro (robot description, xacro)
@@ -32,5 +32,19 @@
     <child link="laser" />
   </joint>
- <link name="usb_cam">
+  <link name="imu_link">
+      <visual>
+        <origin xyz="0 0 0" rpy="0 0 0" />
+        <geometry>
+          <box size="0.01 0.01 0.01" />
+        </geometry>
+        <material name="Grey" />
+      </visual>
+  </link>
+  <joint name="base_link_to_imu_link" type="fixed">
+    <origin xyz="0.0 0 0.2" rpy="0 0 0" />
+    <parent link="base_link"/>
+    <child link="imu_link" />
+  </joint>
+  <link name="usb_cam">
       <visual>
         <origin xyz="0 0 0" rpy="0 0 0" />
